File: schematics/ControlLogic.sch (KiCad schematic (older format))
At the start: 22 parts

Commit message: rearrange outputs of microcode eeproms
Parts:
- removed U? (x4): 74LS04, symbol 74xx:74LS04
- added U? (x2): 74LS137, symbol 74xx:74LS137
- added U? (x9): 74LS04, symbol 74xx:74LS04
Connections:
- net +5V: now also U?.16 (VCC), U?.6 (G1)
- net AddressLatch_IN: now also U?.2
- net DataBuffer_IN: now also U?.6
- net Flashs/D14: now also U?.1 (A0); no longer U?.3
- net Flashs/D15: now also U?.2 (A1); no longer U?.5
- net Flashs/D16: now also U?.3 (A2); no longer U?.9
- net Flashs/D17: now also U?.3; no longer U?.11
- net Flashs/D18: now also U?.5; no longer U?.13
- net Flashs/D19: now also U?.9; no longer U?.1
- net Flashs/D20: now also U?.11; no longer U?.3
- net Flashs/D21: now also U?.13; no longer U?.5
- net Flashs/D22: now also U?.1
- net Flashs/D23: now also U?.3
- net Flashs/D24: now also U?.5
- net Flashs/D38: no longer U?.4 (D1)
- net Flashs/D39: no longer U?.5 (D2)
- net Flashs/D40: no longer U?.6 (D3)
- net Flashs/D41: no longer U?.1 (A0), U?.1 (A0)
- net Flashs/D42: no longer U?.2 (A1), U?.2 (A1)
- net Flashs/D43: no longer U?.3 (A2), U?.3 (A2)
- net Flashs/D44: no longer U?.5 (~G2), U?.6 (G1)
- net Flashs/D45: no longer U?.1 (A0)
- net Flashs/D46: no longer U?.2 (A1)
- net Flashs/D47: no longer U?.3 (A2)
- net GND: now also U?.4 (~GL), U?.4 (~GL), U?.5 (~G2), U?.8 (GND), U?.8 (GND)
- net InstructionRegister_IN: now also U?.4
- net RegisterA_IN: now also U?.2
- net RegisterB_IN: now also U?.4
- net RegisterC_IN: now also U?.6
- net RegisterD_IN: now also U?.8
- net RegisterW_IN: now also U?.10
- net RegisterZ_IN: now also U?.12
- net ~ProgramCounter_IN: now also U?.9 (Y6); no longer U?.10
- net ~ProgramCounter_OUT_ADDRESS: now also U?.12 (Y3); no longer U?.14 (Y1)
- net ~RegisterX_COUNT_DOWN: now also U?.6
- net ~RegisterX_COUNT_UP: now also U?.4; no longer U?.6
- net ~RegisterX_IN: now also U?.11 (Y4); no longer U?.4
- net ~RegisterX_OUT_ADDRESS: now also U?.14 (Y1); no longer U?.12 (Y3)
- net ~RegisterY_COUNT_DOWN: now also U?.10
- net ~RegisterY_COUNT_UP: now also U?.8
- net ~RegisterY_IN: now also U?.10 (Y5)
- net ~RegisterY_OUT_ADDRESS: now also U?.13 (Y2); no longer U?.11 (Y4)
- net ~StackPointer_COUNT_DOWN: now also U?.6; no longer U?.8
- net ~StackPointer_COUNT_UP: now also U?.4; no longer U?.6
- net ~StackPointer_IN: now also U?.7 (Y7); no longer U?.4
- net ~StackPointer_OUT_ADDRESS: now also U?.11 (Y4); no longer U?.13 (Y2)
- net Flashs/D0 renamed Flashs/D1
- net Flashs/D37 renamed Flashs/D2
- new net: U?.11 (Y4), U?.5
- new net: U?.12 (Y3), U?.3
- new net: U?.1, U?.13 (Y2)
- new net: U?.13, U?.14 (Y1)
- new net: U?.11, U?.15 (Y0)
- new net: U?.12 (Y3), U?.9
- new net: U?.13 (Y2), U?.5
- new net: U?.14 (Y1), U?.3
- new net: U?.1, U?.15 (Y0)
- new net Flashs/D10: U?.1 (A0), U?.1 (A0)
- new net Flashs/D11: U?.2 (A1), U?.2 (A1)
- new net Flashs/D12: U?.3 (A2), U?.3 (A2)
- new net Flashs/D13: U?.5 (~G2), U?.6 (G1)
- new net Flashs/D3: U?.4 (D1)
- new net Flashs/D4: U?.5 (D2)
- new net Flashs/D5: U?.6 (D3)
- new net Flashs/D6: U?.1 (A0), U?.1 (A0)
- new net Flashs/D7: U?.2 (A1), U?.2 (A1)
- new net Flashs/D8: U?.3 (A2), U?.3 (A2)
- new net Flashs/D9: U?.5 (~G2), U?.6 (G1)
Other:
- moved on the sheet: U?, U?A, U?B, U?C, U?D, U?E, U?F

Commit message: update schematics
Parts:
- removed U?: 74LS157, symbol 74xx:74LS157
- removed U? (x2): 74LS04, symbol 74xx:74LS04
- removed U? (x3): 74LS32, symbol 74xx:74LS32
- added U?: 74LS151, symbol 74xx:74LS151
- added U? (x2): 74LS32, symbol 74xx:74LS32
- added U?: 74LS04, symbol 74xx:74LS04
- added U? (x2): 74LS86, symbol 74xx:74LS86
Connections:
- net Flashs/D5 is gone; now on net GND: U?.6 (D3)
- net +5V: now also U?.16 (VCC), U?.4 (I0)
- net CARRY_FLAG: now also U?.1, U?.2 (I2)
- net DataBuffer_IN: now also U?.4
- net Flashs/A3: now also U?.3; no longer U?.11 (Q3)
- net INSTRUCTION_0: now also U?.1
- net INSTRUCTION_1: now also U?.11 (S0)
- net INSTRUCTION_2: now also U?.10 (S1)
- net INSTRUCTION_3: now also U?.9 (S2)
- net InstructionRegister_IN: no longer U?.4
- net NEGATIVE_FLAG: now also U?.1, U?.1 (I3)
- net OVERFLOW_FLAG: now also U?.15 (I4), U?.2
- net ZERO_FLAG: now also U?.2, U?.2, U?.3 (I1)
- new net: U?.12 (I7), U?.3
- new net: U?.1, U?.13 (I6), U?.3
- new net: U?.14 (I5), U?.3
- new net: U?.2, U?.5 (Z)
- new net: U?.1, U?.2
Other:
- moved on the sheet: U?, U?A, U?B, U?C, U?D, U?E, U?F

Commit message: update schematics
Parts:
- removed U?: 74LS04, symbol 74xx:74LS04
- added U? (x2): 74LS86, symbol 74xx:74LS86
Connections:
- net +5V: now also U?.2
- net CARRY_FLAG: now also U?.1
- net GND: now also U?.7 (~E), U?.8 (GND)
- net at U?.1: now also U?.3
- net DataBuffer_IN: no longer names the net of U?.4
- net DataBuffer_IN: now also U?.1
- net ~DataBuffer_OUT renamed DataBuffer_DIR
- net DataBuffer_DIR: now also U?.2
- new net ~DataBuffer_ENABLE: U?.3
Changed lines of the file:
@@
 	0    1    1    0
 $EndComp
-Text HLabel 3350 4300 0    50   Input ~ 0
-OVERFLOW_FLAG
-Text HLabel 3350 4200 0    50   Input ~ 0
-NEGATIVE_FLAG
-Text HLabel 3350 4100 0    50   Input ~ 0
-CARRY_FLAG
-Text HLabel 3350 4000 0    50   Input ~ 0
-ZERO_FLAG
 Wire Wire Line
 	5750 3950 5750 4000
@@
 	1    0    0    -1
 $EndComp
-Text GLabel 13550 5900 2    50   Output ~ 0
-~DataBuffer_OUT
 Entry Wire Line
 	5900 6200 6000 6300
@@
 	13150 6050 13550 6050
 Wire Wire Line
-	13550 5900 13200 5900
-Wire Wire Line
-	13200 5900 13200 5550
-Wire Wire Line
 	13200 5550 12950 5550
 Wire Wire Line
@@
 Text GLabel 14500 2300 2    50   Output ~ 0
 RegisterW_IN
-Text GLabel 14500 1400 2    50   Output ~ 0
-DataBuffer_IN
 Text GLabel 14500 1700 2    50   Output ~ 0
 AddressLatch_IN
@@
 	1    0    0    -1
 $EndComp
-$Comp
-L 74xx:74LS32 U?
-U 1 1 605DEE98
-P 2150 3600
-F 0 "U?" H 2150 3925 50  0000 C CNN
-F 1 "74LS32" H 2150 3834 50  0000 C CNN
-F 2 "" H 2150 3600 50  0001 C CNN
-F 3 "http://www.ti.com/lit/gpn/sn74LS32" H 2150 3600 50  0001 C CNN
-	1    2150 3600
-	1    0    0    -1
-$EndComp
-$Comp
-L 74xx:74LS04 U?
-U 1 1 605E2238
-P 1550 3500
-F 0 "U?" H 1550 3817 50  0000 C CNN
-F 1 "74LS04" H 1550 3726 50  0000 C CNN
-F 2 "" H 1550 3500 50  0001 C CNN
-F 3 "http://www.ti.com/lit/gpn/sn74LS04" H 1550 3500 50  0001 C CNN
-	1    1550 3500
-	1    0    0    -1
-$EndComp
-$Comp
-L 74xx:74LS86 U?
-U 1 1 6062D5CF
-P 2150 4000
-F 0 "U?" H 2150 4325 50  0000 C CNN
-F 1 "74LS86" H 2150 4234 50  0000 C CNN
-F 2 "" H 2150 4000 50  0001 C CNN
-F 3 "74xx/74ls86.pdf" H 2150 4000 50  0001 C CNN
-	1    2150 4000
-	1    0    0    -1
-$EndComp
-$Comp
-L 74xx:74LS32 U?
-U 1 1 6062F278
-P 2150 4400
-F 0 "U?" H 2150 4725 50  0000 C CNN
-F 1 "74LS32" H 2150 4634 50  0000 C CNN
-F 2 "" H 2150 4400 50  0001 C CNN
-F 3 "http://www.ti.com/lit/gpn/sn74LS32" H 2150 4400 50  0001 C CNN
-	1    2150 4400
-	1    0    0    -1
-$EndComp
-Wire Wire Line
-	2450 4000 2550 4000
-Wire Wire Line
-	2550 4000 2550 4200
-Wire Wire Line
-	2550 4200 1750 4200
-Wire Wire Line
-	1750 4200 1750 4300
-Wire Wire Line
-	1750 4300 1850 4300
-Wire Wire Line
-	1850 4500 1700 4500
-Wire Wire Line
-	1700 4500 1700 3700
-Wire Wire Line
-	1700 3700 1850 3700
-Wire Wire Line
-	1150 3100 1150 3500
-Wire Wire Line
-	1150 3500 1250 3500
-Wire Wire Line
-	1100 3050 1100 3700
-Wire Wire Line
-	1100 3700 1700 3700
-Connection ~ 1700 3700
-Wire Wire Line
-	3350 4000 3450 4000
-Wire Wire Line
-	3350 4100 3400 4100
-Wire Wire Line
-	3350 4200 3500 4200
-Wire Wire Line
-	3350 4300 3550 4300
-Wire Wire Line
-	2550 4200 2550 4500
-Wire Wire Line
-	2550 4500 3600 4500
-Connection ~ 2550 4200
-Wire Wire Line
-	2600 3600 2600 4400
-Wire Wire Line
-	2600 4400 3600 4400
-Wire Wire Line
-	2450 3600 2600 3600
-Wire Wire Line
-	2450 4400 2500 4400
-Wire Wire Line
-	2500 4400 2500 4600
-Wire Wire Line
-	2500 4600 3600 4600
-Wire Wire Line
-	1150 3100 3400 3100
 Wire Wire Line
 	3400 3100 3400 4100
-Connection ~ 3400 4100
 Wire Wire Line
 	3400 4100 3600 4100
@@
 	3450 4000 3450 3050
 Wire Wire Line
-	3450 3050 1100 3050
-Connection ~ 3450 4000
-Wire Wire Line
 	3450 4000 3600 4000
 Wire Wire Line
 	3500 4200 3500 3000
 Wire Wire Line
-	3500 3000 1050 3000
-Wire Wire Line
-	1050 3000 1050 3900
-Wire Wire Line
-	1050 3900 1850 3900
-Connection ~ 3500 4200
-Wire Wire Line
 	3500 4200 3600 4200
 Wire Wire Line
 	3550 4300 3550 2950
-Wire Wire Line
-	3550 2950 1000 2950
-Wire Wire Line
-	1000 2950 1000 4100
-Wire Wire Line
-	1000 4100 1850 4100
-Connection ~ 3550 4300
 Wire Wire Line
 	3550 4300 3600 4300
@@
 	2500 5850 5900 5850
 Connection ~ 5900 5850
+$Comp
+L power:GND #PWR?
+U 1 1 605A32AB
+P 4100 5500
+F 0 "#PWR?" H 4100 5250 50  0001 C CNN
+F 1 "GND" H 4105 5327 50  0000 C CNN
+F 2 "" H 4100 5500 50  0001 C CNN
+F 3 "" H 4100 5500 50  0001 C CNN
+	1    4100 5500
+	1    0    0    -1
+$EndComp
+$Comp
+L power:GND #PWR?
+U 1 1 605C8600
+P 3600 5200
+F 0 "#PWR?" H 3600 4950 50  0001 C CNN
+F 1 "GND" H 3605 5027 50  0000 C CNN
+F 2 "" H 3600 5200 50  0001 C CNN
+F 3 "" H 3600 5200 50  0001 C CNN
+	1    3600 5200
+	0    1    1    0
+$EndComp
+$Comp
+L power:+5V #PWR?
+U 1 1 606961A9
+P 1250 3600
+F 0 "#PWR?" H 1250 3450 50  0001 C CNN
+F 1 "+5V" H 1265 3773 50  0000 C CNN
+F 2 "" H 1250 3600 50  0001 C CNN
+F 3 "" H 1250 3600 50  0001 C CNN
+	1    1250 3600
+	1    0    0    -1
+$EndComp
+Wire Wire Line
+	1150 3400 1250 3400
+Wire Wire Line
+	1150 3100 1150 3400
+$Comp
+L 74xx:74LS86 U?
+U 1 1 6067B100
+P 1550 3500
+F 0 "U?" H 1550 3825 50  0000 C CNN
+F 1 "74LS86" H 1550 3734 50  0000 C CNN
+F 2 "" H 1550 3500 50  0001 C CNN
+F 3 "74xx/74ls86.pdf" H 1550 3500 50  0001 C CNN
+	1    1550 3500
+	1    0    0    -1
+$EndComp
+Wire Wire Line
+	1000 4100 1850 4100
+Wire Wire Line
+	1000 2950 1000 4100
+Wire Wire Line
+	1050 3900 1850 3900
+Wire Wire Line
+	1050 3000 1050 3900
+Wire Wire Line
+	2500 4400 2500 4600
+Wire Wire Line
+	2450 4400 2500 4400
+Wire Wire Line
+	2450 3600 2600 3600
+Wire Wire Line
+	2600 3600 2600 4400
+Connection ~ 2550 4200
+Wire Wire Line
+	2550 4200 2550 4500
+Connection ~ 1700 3700
+Wire Wire Line
+	1100 3700 1700 3700
+Wire Wire Line
+	1100 3050 1100 3700
+Wire Wire Line
+	1700 3700 1850 3700
+Wire Wire Line
+	1700 4500 1700 3700
+Wire Wire Line
+	1850 4500 1700 4500
+Wire Wire Line
+	1750 4300 1850 4300
+Wire Wire Line
+	1750 4200 1750 4300
+Wire Wire Line
+	2550 4200 1750 4200
+Wire Wire Line
+	2550 4000 2550 4200
+Wire Wire Line
+	2450 4000 2550 4000
+$Comp
+L 74xx:74LS32 U?
+U 1 1 6062F278
+P 2150 4400
+F 0 "U?" H 2150 4725 50  0000 C CNN
+F 1 "74LS32" H 2150 4634 50  0000 C CNN
+F 2 "" H 2150 4400 50  0001 C CNN
+F 3 "http://www.ti.com/lit/gpn/sn74LS32" H 2150 4400 50  0001 C CNN
+	1    2150 4400
+	1    0    0    -1
+$EndComp
+$Comp
+L 74xx:74LS86 U?
+U 1 1 6062D5CF
+P 2150 4000
+F 0 "U?" H 2150 4325 50  0000 C CNN
+F 1 "74LS86" H 2150 4234 50  0000 C CNN
+F 2 "" H 2150 4000 50  0001 C CNN
+F 3 "74xx/74ls86.pdf" H 2150 4000 50  0001 C CNN
+	1    2150 4000
+	1    0    0    -1
+$EndComp
+$Comp
+L 74xx:74LS32 U?
+U 1 1 605DEE98
+P 2150 3600
+F 0 "U?" H 2150 3925 50  0000 C CNN
+F 1 "74LS32" H 2150 3834 50  0000 C CNN
+F 2 "" H 2150 3600 50  0001 C CNN
+F 3 "http://www.ti.com/lit/gpn/sn74LS32" H 2150 3600 50  0001 C CNN
+	1    2150 3600
+	1    0    0    -1
+$EndComp
+Wire Wire Line
+	3550 2950 1000 2950
+Wire Wire Line
+	3500 3000 1050 3000
+Wire Wire Line
+	3450 3050 1100 3050
+Wire Wire Line
+	1150 3100 3400 3100
+Wire Wire Line
+	2500 4600 3600 4600
+Wire Wire Line
+	2600 4400 3600 4400
+Wire Wire Line
+	2550 4500 3600 4500
+Connection ~ 3550 4300
+Wire Wire Line
+	3350 4300 3550 4300
+Connection ~ 3500 4200
+Wire Wire Line
+	3350 4200 3500 4200
+Connection ~ 3400 4100
+Wire Wire Line
+	3350 4100 3400 4100
+Connection ~ 3450 4000
+Wire Wire Line
+	3350 4000 3450 4000
+Text HLabel 3350 4000 0    50   Input ~ 0
+ZERO_FLAG
+Text HLabel 3350 4100 0    50   Input ~ 0
+CARRY_FLAG
+Text HLabel 3350 4200 0    50   Input ~ 0
+NEGATIVE_FLAG
+Text HLabel 3350 4300 0    50   Input ~ 0
+OVERFLOW_FLAG
+$Comp
+L 74xx:74LS86 U?
+U 1 1 60834FE3
+P 14800 5150
+F 0 "U?" H 14800 5475 50  0000 C CNN
+F 1 "74LS86" H 14800 5384 50  0000 C CNN
+F 2 "" H 14800 5150 50  0001 C CNN
+F 3 "74xx/74ls86.pdf" H 14800 5150 50  0001 C CNN
+	1    14800 5150
+	1    0    0    -1
+$EndComp
+Wire Wire Line
+	14450 5050 14500 5050
+Text GLabel 15100 5150 2    50   Output ~ 0
+~DataBuffer_ENABLE
+Text GLabel 14600 5400 2    50   Output ~ 0
+DataBuffer_DIR
+Wire Wire Line
+	14600 5400 14500 5400
+Wire Wire Line
+	14500 5400 14500 5250
+Connection ~ 14500 5250
+Wire Wire Line
+	14500 1400 15600 1400
+Wire Wire Line
+	15600 1400 15600 4650
+Wire Wire Line
+	15600 4650 14450 4650
+Wire Wire Line
+	14450 4650 14450 5050
+Wire Wire Line
+	13200 5550 13200 5250
+Wire Wire Line
+	13200 5250 14500 5250
 Wire Bus Line
 	2500 4700 2500 5850
