File: schematics/kicad-project/ControlLogic.sch (KiCad schematic (older format))
At the start: 30 parts

Commit message: Add base pointer register
Parts:
- added U?: 74LS04, symbol 74xx:74LS04
Connections:
- net ~ProgramCounter_IN: now also U?.7 (Y7); no longer U?.9 (Y6)
- net ~RegisterX_IN: now also U?.10 (Y5); no longer U?.11 (Y4)
- net ~RegisterY_IN: now also U?.9 (Y6); no longer U?.10 (Y5)
- net ~StackPointer_IN: now also U?.15 (Y0); no longer U?.7 (Y7)
- net ~BasePointer_OUT_ADDRESS: now reaches U?.9 (Y6)
- net ~BasePointer_OUT_DATA: now reaches U?.11 (Y4)
- net at U?.10 (Y5): now also U?.5
- net at U?.11 (Y4): now also U?.3
- net at U?.12 (Y3): now also U?.1; no longer U?.3
- net at U?.13 (Y2): now also U?.13; no longer U?.1
- net at U?.14 (Y1): now also U?.11; no longer U?.13
- net at U?.9: now also U?.11 (Y4); no longer U?.12 (Y3)
- net at U?.5: now also U?.12 (Y3); no longer U?.13 (Y2)
- net at U?.3: now also U?.13 (Y2); no longer U?.14 (Y1)
- net at U?.1: now also U?.14 (Y1); no longer U?.15 (Y0)
- new net BasePointer_IN: U?.6
Other:
- moved on the sheet: U?A, U?B, U?C, U?D, U?E, U?F
Changed lines of the file:
@@
 $Descr A3 16535 11693
 encoding utf-8
-Sheet 7 24
+Sheet 7 25
 Title ""
 Date ""
@@
 	1    0    0    -1
 $EndComp
-Text GLabel 14500 2550 2    50   Output ~ 0
+Text GLabel 14500 2450 2    50   Output ~ 0
 ~StackPointer_IN
-Text GLabel 14500 2700 2    50   Output ~ 0
+Text GLabel 14500 2600 2    50   Output ~ 0
 ~ProgramCounter_IN
-Text GLabel 14500 2850 2    50   Output ~ 0
+Text GLabel 14500 2750 2    50   Output ~ 0
 ~RegisterY_IN
-Text GLabel 14500 4200 2    50   Output ~ 0
+Text GLabel 14500 4100 2    50   Output ~ 0
 RegisterA_IN
-Text GLabel 14500 3900 2    50   Output ~ 0
+Text GLabel 14500 3800 2    50   Output ~ 0
 RegisterB_IN
-Text GLabel 14500 3600 2    50   Output ~ 0
+Text GLabel 14500 3500 2    50   Output ~ 0
 RegisterC_IN
-Text GLabel 14500 3300 2    50   Output ~ 0
+Text GLabel 14500 3200 2    50   Output ~ 0
 RegisterD_IN
-Text GLabel 14500 3000 2    50   Output ~ 0
+Text GLabel 14500 2900 2    50   Output ~ 0
 ~RegisterX_IN
 $Comp
 L 74xx:74LS04 U?
 U 1 1 5FFE0A94
-P 14200 4200
-F 0 "U?" H 14200 4517 50  0000 C CNN
-F 1 "74LS04" H 14200 4426 50  0000 C CNN
-F 2 "" H 14200 4200 50  0001 C CNN
-F 3 "http://www.ti.com/lit/gpn/sn74LS04" H 14200 4200 50  0001 C CNN
-	1    14200 4200
+P 14200 4100
+F 0 "U?" H 14200 4417 50  0000 C CNN
+F 1 "74LS04" H 14200 4326 50  0000 C CNN
+F 2 "" H 14200 4100 50  0001 C CNN
+F 3 "http://www.ti.com/lit/gpn/sn74LS04" H 14200 4100 50  0001 C CNN
+	1    14200 4100
 	1    0    0    -1
 $EndComp
@@
 L 74xx:74LS04 U?
 U 2 1 5FFE2E6B
-P 14200 3900
-F 0 "U?" H 14200 4217 50  0000 C CNN
-F 1 "74LS04" H 14200 4126 50  0000 C CNN
-F 2 "" H 14200 3900 50  0001 C CNN
-F 3 "http://www.ti.com/lit/gpn/sn74LS04" H 14200 3900 50  0001 C CNN
-	2    14200 3900
+P 14200 3800
+F 0 "U?" H 14200 4117 50  0000 C CNN
+F 1 "74LS04" H 14200 4026 50  0000 C CNN
+F 2 "" H 14200 3800 50  0001 C CNN
+F 3 "http://www.ti.com/lit/gpn/sn74LS04" H 14200 3800 50  0001 C CNN
+	2    14200 3800
 	1    0    0    -1
 $EndComp
@@
 L 74xx:74LS04 U?
 U 3 1 5FFEF2FB
-P 14200 3600
-F 0 "U?" H 14200 3917 50  0000 C CNN
-F 1 "74LS04" H 14200 3826 50  0000 C CNN
-F 2 "" H 14200 3600 50  0001 C CNN
-F 3 "http://www.ti.com/lit/gpn/sn74LS04" H 14200 3600 50  0001 C CNN
-	3    14200 3600
+P 14200 3500
+F 0 "U?" H 14200 3817 50  0000 C CNN
+F 1 "74LS04" H 14200 3726 50  0000 C CNN
+F 2 "" H 14200 3500 50  0001 C CNN
+F 3 "http://www.ti.com/lit/gpn/sn74LS04" H 14200 3500 50  0001 C CNN
+	3    14200 3500
 	1    0    0    -1
 $EndComp
@@
 L 74xx:74LS04 U?
 U 4 1 5FFF125A
-P 14200 3300
-F 0 "U?" H 14200 3617 50  0000 C CNN
-F 1 "74LS04" H 14200 3526 50  0000 C CNN
-F 2 "" H 14200 3300 50  0001 C CNN
-F 3 "http://www.ti.com/lit/gpn/sn74LS04" H 14200 3300 50  0001 C CNN
-	4    14200 3300
+P 14200 3200
+F 0 "U?" H 14200 3517 50  0000 C CNN
+F 1 "74LS04" H 14200 3426 50  0000 C CNN
+F 2 "" H 14200 3200 50  0001 C CNN
+F 3 "http://www.ti.com/lit/gpn/sn74LS04" H 14200 3200 50  0001 C CNN
+	4    14200 3200
 	1    0    0    -1
 $EndComp
@@
 L 74xx:74LS04 U?
 U 5 1 5FFF3373
-P 14200 2300
-F 0 "U?" H 14200 2617 50  0000 C CNN
-F 1 "74LS04" H 14200 2526 50  0000 C CNN
-F 2 "" H 14200 2300 50  0001 C CNN
-F 3 "http://www.ti.com/lit/gpn/sn74LS04" H 14200 2300 50  0001 C CNN
-	5    14200 2300
+P 14200 2200
+F 0 "U?" H 14200 2517 50  0000 C CNN
+F 1 "74LS04" H 14200 2426 50  0000 C CNN
+F 2 "" H 14200 2200 50  0001 C CNN
+F 3 "http://www.ti.com/lit/gpn/sn74LS04" H 14200 2200 50  0001 C CNN
+	5    14200 2200
 	1    0    0    -1
 $EndComp
@@
 L 74xx:74LS04 U?
 U 6 1 5FFF5245
-P 14200 2000
-F 0 "U?" H 14200 2317 50  0000 C CNN
-F 1 "74LS04" H 14200 2226 50  0000 C CNN
-F 2 "" H 14200 2000 50  0001 C CNN
-F 3 "http://www.ti.com/lit/gpn/sn74LS04" H 14200 2000 50  0001 C CNN
-	6    14200 2000
-	1    0    0    -1
-$EndComp
-Wire Wire Line
-	12950 4200 13900 4200
-Wire Wire Line
-	12950 4100 13700 4100
-Wire Wire Line
-	13700 4100 13700 3900
-Wire Wire Line
-	13700 3900 13900 3900
-Wire Wire Line
-	12950 4000 13650 4000
-Wire Wire Line
-	13650 4000 13650 3600
-Wire Wire Line
-	13650 3600 13900 3600
-Wire Wire Line
-	12950 3900 13600 3900
-Wire Wire Line
-	13600 3900 13600 3300
-Wire Wire Line
-	13600 3300 13900 3300
-Wire Wire Line
-	12950 3800 13550 3800
-Wire Wire Line
-	12950 3700 13500 3700
+P 14200 1900
+F 0 "U?" H 14200 2217 50  0000 C CNN
+F 1 "74LS04" H 14200 2126 50  0000 C CNN
+F 2 "" H 14200 1900 50  0001 C CNN
+F 3 "http://www.ti.com/lit/gpn/sn74LS04" H 14200 1900 50  0001 C CNN
+	6    14200 1900
+	1    0    0    -1
+$EndComp
+Wire Wire Line
+	12950 4100 13900 4100
+Wire Wire Line
+	12950 4000 13700 4000
+Wire Wire Line
+	13700 4000 13700 3800
+Wire Wire Line
+	13700 3800 13900 3800
+Wire Wire Line
+	12950 3900 13650 3900
+Wire Wire Line
+	13650 3900 13650 3500
+Wire Wire Line
+	13650 3500 13900 3500
+Wire Wire Line
+	12950 3800 13600 3800
+Wire Wire Line
+	13600 3800 13600 3200
+Wire Wire Line
+	13600 3200 13900 3200
+Wire Wire Line
+	12950 3700 13550 3700
+Wire Wire Line
+	12950 3600 13500 3600
 $Comp
 L 74xx:74LS04 U?
 U 1 1 600BF50B
-P 14200 1700
-F 0 "U?" H 14200 2017 50  0000 C CNN
-F 1 "74LS04" H 14200 1926 50  0000 C CNN
-F 2 "" H 14200 1700 50  0001 C CNN
-F 3 "http://www.ti.com/lit/gpn/sn74LS04" H 14200 1700 50  0001 C CNN
-	1    14200 1700
+P 14200 1600
+F 0 "U?" H 14200 1917 50  0000 C CNN
+F 1 "74LS04" H 14200 1826 50  0000 C CNN
+F 2 "" H 14200 1600 50  0001 C CNN
+F 3 "http://www.ti.com/lit/gpn/sn74LS04" H 14200 1600 50  0001 C CNN
+	1    14200 1600
 	1    0    0    -1
 $EndComp
@@
 L 74xx:74LS04 U?
 U 2 1 600BF511
-P 14200 1400
-F 0 "U?" H 14200 1717 50  0000 C CNN
-F 1 "74LS04" H 14200 1626 50  0000 C CNN
-F 2 "" H 14200 1400 50  0001 C CNN
-F 3 "http://www.ti.com/lit/gpn/sn74LS04" H 14200 1400 50  0001 C CNN
-	2    14200 1400
-	1    0    0    -1
-$EndComp
-Wire Wire Line
-	12950 3600 13450 3600
-Wire Wire Line
-	12950 3500 13400 3500
-Wire Wire Line
-	12950 2350 13250 2350
-Wire Wire Line
-	13250 2350 13250 1700
-Wire Wire Line
-	13250 1700 13900 1700
-Wire Wire Line
-	12950 2250 13200 2250
-Wire Wire Line
-	13200 2250 13200 1400
-Wire Wire Line
-	13200 1400 13900 1400
+P 14200 1300
+F 0 "U?" H 14200 1617 50  0000 C CNN
+F 1 "74LS04" H 14200 1526 50  0000 C CNN
+F 2 "" H 14200 1300 50  0001 C CNN
+F 3 "http://www.ti.com/lit/gpn/sn74LS04" H 14200 1300 50  0001 C CNN
+	2    14200 1300
+	1    0    0    -1
+$EndComp
+Wire Wire Line
+	12950 3500 13450 3500
+Wire Wire Line
+	12950 2250 13250 2250
+Wire Wire Line
+	13250 2250 13250 1600
+Wire Wire Line
+	13250 1600 13900 1600
+Wire Wire Line
+	12950 2150 13200 2150
+Wire Wire Line
+	13200 2150 13200 1300
+Wire Wire Line
+	13200 1300 13900 1300
 Wire Wire Line
 	5650 2700 5650 3300
@@
 	13100 6200 13550 6200
 Wire Wire Line
-	13550 3800 13550 3000
-Wire Wire Line
-	13550 3000 14500 3000
-Wire Wire Line
-	14500 2850 13500 2850
-Wire Wire Line
-	13500 2850 13500 3700
-Wire Wire Line
-	13450 2700 14500 2700
-Wire Wire Line
-	13450 2700 13450 3600
-Wire Wire Line
-	14500 2550 13400 2550
-Wire Wire Line
-	13400 2550 13400 3500
-Wire Wire Line
-	12950 2450 13300 2450
-Wire Wire Line
-	13300 2450 13300 2000
-Wire Wire Line
-	13300 2000 13900 2000
-Wire Wire Line
-	12950 2550 13350 2550
-Wire Wire Line
-	13350 2550 13350 2300
-Wire Wire Line
-	13350 2300 13900 2300
-Text GLabel 14500 2000 2    50   Output ~ 0
+	13550 3700 13550 2900
+Wire Wire Line
+	13550 2900 14500 2900
+Wire Wire Line
+	14500 2750 13500 2750
+Wire Wire Line
+	13500 2750 13500 3600
+Wire Wire Line
+	13450 2600 14500 2600
+Wire Wire Line
+	13450 2600 13450 3500
+Wire Wire Line
+	14500 2450 13400 2450
+Wire Wire Line
+	12950 2350 13300 2350
+Wire Wire Line
+	13300 2350 13300 1900
+Wire Wire Line
+	13300 1900 13900 1900
+Wire Wire Line
+	12950 2450 13350 2450
+Wire Wire Line
+	13350 2450 13350 2200
+Wire Wire Line
+	13350 2200 13900 2200
+Text GLabel 14500 1900 2    50   Output ~ 0
 RegisterZ_IN
-Text GLabel 14500 2300 2    50   Output ~ 0
+Text GLabel 14500 2200 2    50   Output ~ 0
 RegisterW_IN
-Text GLabel 14500 1700 2    50   Output ~ 0
+Text GLabel 14500 1600 2    50   Output ~ 0
 AddressLatch_IN
 Text GLabel 7550 5000 2    50   Output ~ 0
@@
 Connection ~ 14500 5250
 Wire Wire Line
-	14500 1400 15600 1400
-Wire Wire Line
-	15600 1400 15600 4650
+	14500 1300 15600 1300
 Wire Wire Line
 	15600 4650 14450 4650
@@
 Wire Wire Line
 	13200 5250 14500 5250
+Wire Wire Line
+	15600 1300 15600 4650
+Wire Wire Line
+	12950 2550 13400 2550
+Wire Wire Line
+	13400 2550 13400 2450
+$Comp
+L 74xx:74LS04 U?
+U 3 1 6169CB9B
+P 14200 1000
+F 0 "U?" H 14200 1317 50  0000 C CNN
+F 1 "74LS04" H 14200 1226 50  0000 C CNN
+F 2 "" H 14200 1000 50  0001 C CNN
+F 3 "http://www.ti.com/lit/gpn/sn74LS04" H 14200 1000 50  0001 C CNN
+	3    14200 1000
+	1    0    0    -1
+$EndComp
+Text GLabel 14500 1000 2    50   Output ~ 0
+BasePointer_IN
+Wire Wire Line
+	13900 1000 13150 1000
+Wire Wire Line
+	13150 1000 13150 2050
+Wire Wire Line
+	13150 2050 12950 2050
+Text GLabel 13400 8300 2    50   Output ~ 0
+~BasePointer_OUT_ADDRESS
+Wire Wire Line
+	13400 8300 13150 8300
+Wire Wire Line
+	13150 8300 13150 8550
+Wire Wire Line
+	13150 8550 12950 8550
+Text GLabel 13550 5900 2    50   Output ~ 0
+~BasePointer_OUT_DATA
+Wire Wire Line
+	13550 5900 13250 5900
+Wire Wire Line
+	13250 5900 13250 5450
+Wire Wire Line
+	13250 5450 12950 5450
 Wire Bus Line
 	2500 4700 2500 5850
