File: schematics/kicad-project/16-bit computer.sch (KiCad schematic (older format))
At the start: 14 parts

Commit message: Update schematics
Parts:
- removed U? (x2): IS61C5128AS-25TLI, Package_SO:TSOP-II-32_21.0x10.2mm_P1.27mm, symbol Memory_RAM:IS61C5128AS-25TLI
- removed U? (x7): 74LS08, symbol 74xx:74LS08
- added RV?: R_POT, symbol Device:R_POT
- added U? (x2): HM62256BLP, Package_DIP:DIP-28_W15.24mm, symbol Memory_RAM:HM62256BLP
- added U? (x6): 74LS11, symbol 74xx:74LS11
- added U? (x3): 74LS32, symbol 74xx:74LS32
- added U? (x2): 74LS04, symbol 74xx:74LS04
Connections:
- net A0: now also DS?.16 (D/~I~), U?.10 (A0), U?.10 (A0)
- net A1: now also U?.4, U?.5, U?.9 (A1), U?.9 (A1)
- net A10: now also U?.10, U?.21 (A10), U?.21 (A10)
- net A11: now also U?.11, U?.23 (A11), U?.23 (A11)
- net A12: now also U?.1, U?.2 (A12), U?.2 (A12)
- net A13: now also U?.2, U?.26 (A13), U?.26 (A13)
- net A14: now also U?.1 (A14), U?.1 (A14), U?.13
- net A2: now also U?.1, U?.8 (A2), U?.8 (A2)
- net A3: now also U?.1, U?.7 (A3), U?.7 (A3)
- net A4: now also U?.2, U?.6 (A4), U?.6 (A4)
- net A5: now also U?.13, U?.5 (A5), U?.5 (A5)
- net A6: now also U?.3, U?.4 (A6), U?.4 (A6)
- net A7: now also U?.3 (A7), U?.3 (A7), U?.4
- net A8: now also U?.25 (A8), U?.25 (A8), U?.5
- net A9: now also U?.24 (A9), U?.24 (A9), U?.9
- net CPU/~R: now also U?.22 (~OE), U?.22 (~OE)
- net CPU/~W: now also DS?.15 (R/~W~), U?.27 (~WE), U?.27 (~WE); no longer U?.7 (WE), U?.7 (WE)
- net D0: now also DS?.4 (DB0), U?.11 (Q0)
- net D1: now also DS?.5 (DB1), U?.12 (Q1)
- net D10: now also U?.13 (Q2)
- net D11: now also U?.15 (Q3)
- net D12: now also U?.16 (Q4)
- net D13: now also U?.17 (Q5)
- net D14: now also U?.18 (Q6)
- net D15: now also U?.19 (Q7)
- net D2: now also DS?.6 (DB2), U?.13 (Q2)
- net D3: now also DS?.7 (DB3), U?.15 (Q3)
- net D4: now also DS?.8 (DB4), U?.16 (Q4)
- net D5: now also DS?.9 (DB5), U?.17 (Q5)
- net D6: now also DS?.10 (DB6), U?.18 (Q6)
- net D7: now also DS?.11 (DB7), U?.19 (Q7)
- net D8: now also U?.11 (Q0)
- net D9: now also U?.12 (Q1)
- net at U?.3: now also U?.20 (~CS), U?.20 (~CS)
- net GND: now reaches U?.10 (A16)
- net GND: now also DS?.19 (LEDA/EL), DS?.2 (GND), U?.10 (A16), U?.11 (A15), U?.11 (A15), U?.24 (GND), U?.24 (GND), U?.6 (A17), U?.6 (A17), U?.9 (A18), U?.9 (A18), RV?.3, U?.14 (GND), U?.14 (GND)
- net at U?.30 (CE), U?.30 (CE): now also U?.2, U?.5
- net +5V: now reaches U?.8 (VCC)
- net +5V: now also DS?.1 (VCC), U?.7 (WE), U?.7 (WE), U?.8 (VCC), U?.28 (VCC), U?.28 (VCC)
- net at DS?.12 (~CS1~): now also U?.6
- net at DS?.13 (~CS2~): now also U?.8
- net ~RST: now reaches DS?.14 (~RST~)
- net ~CLK: now reaches DS?.17 (E)
- net at DS?.18 (VEE): now also DS?.20 (LEDK/EL), RV?.1
- net at DS?.3 (VO): now also RV?.2
- net IO: no longer names the net of U?.2
- net IO: now also U?.1, U?.6
- new net: U?.1, U?.12
- new net: U?.2, U?.6
- new net: U?.13, U?.8
- new net: U?.12, U?.4
- new net: U?.12, U?.3
- new net: U?.2, U?.2
- new net: U?.10, U?.3, U?.5
- new net: U?.6, U?.9
Other:
- moved on the sheet: DS?, U?A
